File: Herz Vibration/Herz-Vibration_Grupo_6.brd (EAGLE design)
At the start: 72.4 x 60.6 mm, 17 parts, among them IC1 AD8574TRUZ-EP, IC2 ADS131M03IPWR, J1 009276006021106

Commit message: Actualización de esquemáticos y PCB.
Connections:
- removed net N$13: IC2.4
- removed net N$24: IC2.5
- removed net N$25: IC2.8
- net GND: now also IC2.4, IC2.5, IC2.8
Routing:
- net GND: track 44.9 -> 55.2 mm, vias 6 -> 8
Other:
- board text added: "ELO 301 2023"
- board text added: "Herz-Vibration"
Changed lines of the file:
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@@
 <wire x1="72.37" y1="58.09" x2="0" y2="58.09" width="0" layer="20"/>
 <wire x1="0" y1="58.09" x2="0" y2="-2.54" width="0" layer="20"/>
+<text x="40.64" y="12.7" size="1.778" layer="25">Herz-Vibration</text>
+<text x="40.64" y="8.89" size="1.778" layer="25">ELO 301 2023</text>
 </plain>
 <attributes>
@@
 <wire x1="27.875" y1="9.125" x2="27.92" y2="9.18" width="0.1" layer="1"/>
 <wire x1="23" y1="9.125" x2="22.92" y2="9.18" width="0.1" layer="1"/>
+<contactref element="IC2" pad="4"/>
+<contactref element="IC2" pad="8"/>
+<contactref element="IC2" pad="5"/>
+<wire x1="42.782" y1="28.265" x2="41.585" y2="28.265" width="0.1" layer="1"/>
+<wire x1="41.585" y1="28.265" x2="41.275" y2="28.575" width="0.1" layer="1"/>
+<via x="39.37" y="30.48" extent="1-16" drill="0.35"/>
+<wire x1="41.275" y1="28.575" x2="39.37" y2="30.48" width="0.1" layer="1"/>
+<wire x1="42.782" y1="28.915" x2="41.615" y2="28.915" width="0.1" layer="1"/>
+<wire x1="41.615" y1="28.915" x2="41.275" y2="28.575" width="0.1" layer="1"/>
+<wire x1="42.782" y1="26.315" x2="41.555" y2="26.315" width="0.1" layer="1"/>
+<wire x1="41.555" y1="26.315" x2="39.37" y2="24.13" width="0.1" layer="1"/>
+<via x="39.37" y="24.13" extent="1-16" drill="0.35"/>
 </signal>
 <signal name="+3V3">
@@
 <wire x1="40" y1="27.31" x2="38.1" y2="29.21" width="0.1" layer="16"/>
 <via x="38.1" y="29.21" extent="1-16" drill="0.35"/>
-<wire x1="38.1" y1="30.48" x2="38.1" y2="29.21" width="0.1" layer="1"/>
-<wire x1="30.48" y1="38.1" x2="38.1" y2="30.48" width="0.1" layer="1"/>
+<wire x1="34.29" y1="34.29" x2="34.29" y2="33.02" width="0.1" layer="1"/>
+<wire x1="34.29" y1="33.02" x2="38.1" y2="29.21" width="0.1" layer="1"/>
+<wire x1="30.082" y1="38.498" x2="34.29" y2="34.29" width="0.1" layer="1"/>
 <wire x1="28.62" y1="38.498" x2="30.082" y2="38.498" width="0.1" layer="1"/>
-<wire x1="30.082" y1="38.498" x2="30.48" y2="38.1" width="0.1" layer="1"/>
 </signal>
 <signal name="+1V">
@@
 <contactref element="M1" pad="CN5-8"/>
 </signal>
-<signal name="N$13">
-<contactref element="IC2" pad="4"/>
-</signal>
-<signal name="N$24">
-<contactref element="IC2" pad="5"/>
-</signal>
-<signal name="N$25">
-<contactref element="IC2" pad="8"/>
-</signal>
 <signal name="N$27">
